File: daughterboardv4.kicad_sch (KiCad schematic)
At the start: 8 parts, among them J1 DF30FC-24DP-0.4V_81_, U1 TXS0104EBQAR, U2 NCP170AXV180T2G

Commit message: Improved visibility in schematic & pcb
-Added Net Labels for signal channels on both sides of voltage shifter in Schematic Editor
-Arranged footprint silkscreen texts on the board in PCB Editor
Connections:
- net INTERRUPT_EXTI4: now reaches J1.15 (PC4), U1.10 (B4)
- net DFSDM1_CKIN4: now reaches J1.21 (PC1), U1.12 (B2)
- net DFSDM1_DATIN4: now reaches J1.22 (PC0), U1.11 (B3)
- net USART_TX: now reaches J1.7 (PB6), U1.13 (B1)
- net MIC_DATA: now reaches MK1.1 (DATA), U1.4 (A3)
- net MIC_WAKE: now reaches MK1.4 (WAKE), U1.5 (A4)
- net MIC_THSEL: now reaches MK1.5 (THSEL), U1.2 (A1)
- net MIC_CLK: now reaches MK1.6 (CLK), U1.3 (A2)
Changed lines of the file:
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@@
+		)
+	)
+	(label "DFSDM1_DATIN4"
+		(at 96.52 74.93 0)
+		(effects
+			(font
+				(size 1.27 1.27)
+			)
+			(justify left bottom)
+		)
+	)
+	(label "INTERRUPT_EXTI4"
+		(at 95.25 77.47 0)
+		(effects
+			(font
+				(size 1.27 1.27)
+			)
+			(justify left bottom)
+		)
+	)
+	(label "MIC_CLK"
+		(at 158.75 69.85 0)
+		(effects
+			(font
+				(size 1.27 1.27)
+			)
+			(justify left bottom)
+		)
+	)
+	(label "MIC_CLK"
+		(at 158.75 69.85 0)
+		(effects
+			(font
+				(size 1.27 1.27)
+			)
+			(justify left bottom)
+		)
+	)
+	(label "MIC_THSEL"
+		(at 158.75 67.31 0)
+		(effects
+			(font
+				(size 1.27 1.27)
+			)
+			(justify left bottom)
+		)
+	)
+	(label "MIC_DATA"
+		(at 158.75 72.39 0)
+		(effects
+			(font
+				(size 1.27 1.27)
+			)
+			(justify left bottom)
+		)
+	)
+	(label "USART_TX"
+		(at 102.87 69.85 0)
+		(effects
+			(font
+				(size 1.27 1.27)
+			)
+			(justify left bottom)
+		)
+	)
+	(label "MIC_WAKE"
+		(at 158.75 74.93 0)
+		(effects
+			(font
+				(size 1.27 1.27)
+			)
+			(justify left bottom)
+		)
+	)
+	(label "DFSDM1_CKIN4"
+		(at 97.79 72.39 0)
+		(effects
+			(font
+				(size 1.27 1.27)
+			)
+			(justify left bottom)
 		)
 	)
