File: daughterboardv4/daughterboardv4.kicad_pcb (KiCad board)
At the start: 2 copper layers, 8.5 x 10.8 mm, 8 parts, among them J1 DF30FC-24DP-0.4V_81_, U1 TXS0104EBQAR, U2 NCP170AXV180T2G

Commit message: Design updated and optimized (v5)
-Changed voltage level translator from TXS0104E to SN74AVC4T774
-Optimized layout and minimized board dimension to 10.04x7.94mm
-Reorganize projects files into separate versions
Parts:
- U2: value NCP170AXV180T2G -> SOT-563_1P3X1P7_ONS
Changed lines of the file:
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@@
 		)
 		(embedded_fonts no)
-		(model "${KIPRJMOD}/Libraries/ul_TXS0104EBQAR (1)/BQA0014A.stp"
+		(model "${KIPRJMOD}/../Libraries/ul_TXS0104EBQAR (1)/BQA0014A.stp"
 			(offset
 				(xyz 0 0 0)
@@
 			)
 		)
-		(property "Value" "NCP170AXV180T2G"
+		(property "Value" "SOT-563_1P3X1P7_ONS"
 			(at 0 0 0)
 			(unlocked yes)
@@
 			)
 		)
-		(property "Datasheet" "NCP170AXV180T2G"
+		(property "Datasheet" "https://www.onsemi.com/pdf/datasheet/ncp170-d.pdf"
 			(at 0 0 0)
 			(layer "F.Fab")
@@
 		)
 		(embedded_fonts no)
-		(model "${KIPRJMOD}/Libraries/NCP170AXV180T2G/SOT-563_1P3X1P7_ONS.step"
+		(model "${KIPRJMOD}/../Libraries/NCP170AXV180T2G/SOT-563_1P3X1P7_ONS.step"
 			(offset
 				(xyz 0 0 0)
@@
 		)
 		(embedded_fonts no)
-		(model "${KIPRJMOD}/Libraries/SamacSys/SamacSys_Parts.3dshapes/DF30FC-24DP-0.4V_81_.stp"
+		(model "${KIPRJMOD}/../Libraries/SamacSys/SamacSys_Parts.3dshapes/DF30FC-24DP-0.4V_81_.stp"
 			(offset
 				(xyz 0 0 0)
@@
 		)
 		(embedded_fonts no)
-		(model "${KIPRJMOD}/Libraries/MMICT5838_00_012 (2)/MMICT5838-00-012--3DModel-STEP-510211.STEP"
+		(model "${KIPRJMOD}/../Libraries/MMICT5838_00_012 (2)/MMICT5838-00-012--3DModel-STEP-510211.STEP"
 			(offset
 				(xyz 0 0 0)
