File: daughterboardv5/daughterboardv5.kicad_sch (KiCad schematic)
At the start: 8 parts, among them J1 DF30FC-24DP-0.4V_81_, U1 TXS0104EBQAR, U2 NCP170AXV180T2G

Commit message: Design updated and optimized (v5)
-Changed voltage level translator from TXS0104E to SN74AVC4T774
-Optimized layout and minimized board dimension to 10.04x7.94mm
-Reorganize projects files into separate versions
Parts:
- removed U1: TXS0104EBQAR, volshift_TXS0104EBQAR:WQFN14_BQA_TEX, symbol volshift_TXS0104EBQAR:TXS0104EBQAR
- added U1: SN74AVC4T774BQBR, volshift_SN74AVC4T774:BQB0016A-MFG, symbol volshift_SN74AVC4T774:SN74AVC4T774BQBR
Connections:
- net +1V8: now also U1.15 (VCCB)
- net +2V8: now also U1.16 (VCCA), U1.7 (DIR3), U1.8 (DIR4), U1.9 (OE_N)
- net DFSDM1_CKIN4: now also U1.5 (A3)
- net DFSDM1_DATIN4: now also U1.4 (A2)
- net GND: now also U1.1 (DIR1), U1.10 (GND), U1.17 (Thermal_Pad), U1.2 (DIR2)
- net INTERRUPT_EXTI4: now also U1.3 (A1)
- net MIC_CLK: now also U1.12 (B3)
- net MIC_DATA: now also U1.13 (B2)
- net MIC_THSEL: now also U1.11 (B4)
- net MIC_WAKE: now also U1.14 (B1)
- net USART_TX: now also U1.6 (A4)
